Commit message: URDF수정
Gazebo에 적용할 수 있도록 collision 수정..
아직 완성은 아님

File: canDynamix/candynamix_description/urdf/candynamix.urdf.xacro (robot description, xacro)
@@ -7,9 +7,9 @@
     <parent link="base_footprint"/>
     <child link="base_link"/>
-    <origin xyz="0 0 0.0" rpy="0 0 0"/>
+    <origin xyz="0 0 0" rpy="0 0 0"/>
   </joint>
   <link name="base_link">
     <visual>
-      <origin xyz="-0.0345 0.112 0.077" rpy="0 0 3.14"/>
+	<origin xyz="-0.0345 0.112 0.077" rpy="0 0 3.14"/>
       <geometry>
         <mesh filename="package://candynamix_description/meshes/bases/candynamix_base.stl" scale="0.001 0.001 0.001"/>
@@ -18,11 +18,11 @@
     </visual>
     <collision>
-      <origin xyz="-0.0345 0.112 0.077" rpy="0 0 3.14"/>
+      <origin xyz="-0.01 0 0.035" rpy="0 0 0"/>
       <geometry>
-        <box size="0.140 0.140 0.140"/>
+        <cylinder length="0.05" radius="0.06"/>
       </geometry>
     </collision>
     <inertial>
-      <origin xyz="-0.0345 0.112 0.077" rpy="0 0 3.14"/>
+      <origin xyz="0 0 0" rpy="0 0 0"/>
       <mass value="1"/>
       <inertia ixx="0.01" ixy="0.0" ixz="0.0"
@@ -46,7 +46,7 @@
     </visual>
     <collision>
-      <origin xyz="0 0 0" rpy="0 0 0"/>
+      <origin xyz="0 0.005 0" rpy="${-M_PI*0.5} 0 0"/>
       <geometry>
-        <cylinder length="0.018" radius="0.033"/>
+        <cylinder length="0.005" radius="0.018"/>
       </geometry>
     </collision>
@@ -62,5 +62,4 @@
     <parent link="base_link"/>
     <child link="wheel_right_link"/>
-<!-- origin xyz="0 0.036 0.016" rpy="${-M_PI*0.5} 1.57 1.57"/-->
     <origin xyz="0 -0.038 0.016" rpy="${-M_PI*0.5} -1.57 1.57"/>
     <axis xyz="0 1 0"/>
@@ -75,7 +74,7 @@
     </visual>
     <collision>
-      <origin xyz="0 0 0" rpy="0 0 0"/>
+      <origin xyz="0 -0.005 0" rpy="${M_PI*0.5} 0 0"/>
       <geometry>
-        <cylinder length="0.018" radius="0.033"/>
+        <cylinder length="0.005" radius="0.018"/>
       </geometry>
     </collision>
@@ -91,11 +90,11 @@
     <parent link="base_link"/>
     <child link="caster_back_link"/>
-    <origin xyz="-0.081 0 -0.004" rpy="${-M_PI*0.5} 0 0"/>
+    <origin xyz="-0.056 0 0.002" rpy="${-M_PI*0.5} 0 0"/>
   </joint>
   <link name="caster_back_link">
     <collision>
-      <origin xyz="0 0 0" rpy="0 0 0"/>
+      <origin xyz="0 0 0" rpy="${M_PI*0.5} 0 0"/>
       <geometry>
-        <box size="0.030 0.010 0.020"/>
+        <cylinder length="0.005" radius="0.01"/>
       </geometry>
     </collision>
@@ -130,5 +129,5 @@
       <origin xyz="0 0 0" rpy="0 0 0"/>
       <geometry>
-        <cylinder length="0.0408" radius="0.070"/>
+        <cylinder length="0.003" radius="0.003"/>
       </geometry>
     </collision>
