Commit message: base_scan link 추가
HC-SR04-UltrasonicSensor.stl 추가 후 URDF 파일 작성

File: canDynamix/candynamix_description/urdf/candynamix.gazebo.xacro (robot description, xacro)
@@ -1,4 +1,4 @@
 <?xml version="1.0"?>
-<robot name="candynamix_sim" xmlns:xacro="http://ros.org/wiki/xacro">
+<robot name="candynamix" xmlns:xacro="http://ros.org/wiki/xacro">
   <xacro:arg name="laser_visual" default="false"/>
   <xacro:arg name="imu_visual"   default="false"/>

File: canDynamix/candynamix_description/urdf/candynamix.urdf.xacro (robot description, xacro)
@@ -34,5 +34,5 @@
     <parent link="base_link"/>
     <child link="wheel_left_link"/>
-    <origin xyz="0 0.038 0.016" rpy="${M_PI*0.5} 1.58 1.58"/>
+    <origin xyz="0 0.038 0.016" rpy="${M_PI*0.5} 1.57 1.57"/>
     <axis xyz="0 1 0"/>
   </joint>
@@ -62,6 +62,6 @@
     <parent link="base_link"/>
     <child link="wheel_right_link"/>
-<!-- origin xyz="0 0.036 0.016" rpy="${-M_PI*0.5} 1.58 1.58"/-->
-    <origin xyz="0 -0.038 0.016" rpy="${-M_PI*0.5} -1.58 1.58"/>
+<!-- origin xyz="0 0.036 0.016" rpy="${-M_PI*0.5} 1.57 1.57"/-->
+    <origin xyz="0 -0.038 0.016" rpy="${-M_PI*0.5} -1.57 1.57"/>
     <axis xyz="0 1 0"/>
   </joint>
@@ -117,12 +117,11 @@
     <parent link="base_link"/>
     <child link="base_scan"/>
-    <origin xyz="-0.032 0 0.171" rpy="0 0 0"/>
+    <origin xyz="0.03 0 0.03" rpy="${M_PI*0.5} 0 1.57 "/>
   </joint>
   <link name="base_scan">
-<!--
     <visual>
-      <origin xyz="0 0 0.0" rpy="0 0 0"/>
+      <origin xyz="0 0 0" rpy="0 0 0"/>
       <geometry>
-        <mesh filename="package://candynamix/candynamix_description/meshes/sensors/lds.stl" scale="0.001 0.001 0.001"/>
+        <mesh filename="package://candynamix_description/meshes/sensors/HC-SR04-UltrasonicSensor.stl" scale="0.001 0.001 0.001"/>
       </geometry>
       <material name="dark"/>
@@ -141,5 +140,4 @@
                izz="0.001" />
     </inertial>
--->
   </link>
 </robot>

Commit message: gazebo수정
가제보에 적용할 수 있도록 collision수정

File: canDynamix/candynamix_description/urdf/candynamix.gazebo.xacro (robot description, xacro)
@@ -22,5 +22,5 @@
   </gazebo>
   <gazebo reference="base_link">
-    <material>Gazebo/Grey</material>
+    <material><color rgba="${255/255} ${108/255} ${10/255} 1.0"/></material>
   </gazebo>
   <gazebo reference="wheel_left_link">

Commit message: gazebo를 위한 inertia 수정중
가베보를 위한 URDF파일 수정중

File: canDynamix/candynamix_description/urdf/candynamix.gazebo.xacro (robot description, xacro)
@@ -15,6 +15,6 @@
       <leftJoint>wheel_left_joint</leftJoint>
       <rightJoint>wheel_right_joint</rightJoint>
-      <wheelSeparation>0.160</wheelSeparation>
-      <wheelDiameter>0.066</wheelDiameter>
+      <wheelSeparation>0.085</wheelSeparation>
+      <wheelDiameter>0.033</wheelDiameter>
       <wheelAcceleration>1</wheelAcceleration>
       <wheelTorque>10</wheelTorque>

File: canDynamix/candynamix_description/urdf/candynamix.urdf.xacro (robot description, xacro)
@@ -26,7 +26,7 @@
       <origin xyz="0 0 0" rpy="0 0 0"/>
       <mass value="1"/>
-      <inertia ixx="0.01" ixy="0.0" ixz="0.0"
-               iyy="0.01" iyz="0.0"
-               izz="0.01" />
+      <inertia ixx="0.05" ixy="0.0" ixz="0.0"
+               iyy="0.05" iyz="0.0"
+               izz="0.05" />
     </inertial>
   </link>
@@ -54,7 +54,7 @@
       <origin xyz="0 0 0" />
       <mass value="0.01" />
-      <inertia ixx="0.001" ixy="0.0" ixz="0.0"
-               iyy="0.001" iyz="0.0"
-               izz="0.001" />
+      <inertia ixx="0.05" ixy="0.0" ixz="0.0"
+               iyy="0.05" iyz="0.0"
+               izz="0.05" />
     </inertial>
   </link>
@@ -82,7 +82,7 @@
       <origin xyz="0 0 0" />
       <mass value="0.01" />
-      <inertia ixx="0.001" ixy="0.0" ixz="0.0"
-               iyy="0.001" iyz="0.0"
-               izz="0.001" />
+      <inertia ixx="0.05" ixy="0.0" ixz="0.0"
+               iyy="0.05" iyz="0.0"
+               izz="0.05" />
     </inertial>
   </link>
@@ -101,8 +101,8 @@
     <inertial>
       <origin xyz="0 0 0" />
-      <mass value="0.01" />
-      <inertia ixx="0.001" ixy="0.0" ixz="0.0"
-               iyy="0.001" iyz="0.0"
-               izz="0.001" />
+      <mass value="0.1" />
+      <inertia ixx="0.05" ixy="0.0" ixz="0.0"
+               iyy="0.05" iyz="0.0"
+               izz="0.05" />
     </inertial>
   </link>
@@ -135,7 +135,7 @@
       <mass value="0.01" />
       <origin xyz="0 0 0" />
-      <inertia ixx="0.001" ixy="0.0" ixz="0.0"
-               iyy="0.001" iyz="0.0"
-               izz="0.001" />
+      <inertia ixx="0.05" ixy="0.0" ixz="0.0"
+               iyy="0.05" iyz="0.0"
+               izz="0.05" />
     </inertial>
   </link>
