Commit message: lds & picamera stl파일 추가
roslaunch candynamix_bringup candynamix_bringup.launch

roslaunch candynamix_rviz candynamix_rviz.launch

로 확인해 보세요.

File: canDynamix/candynamix_description/urdf/candynamix.gazebo.xacro (robot description, xacro)
@@ -1,138 +1,122 @@
 <?xml version="1.0"?>
 <robot name="candynamix" xmlns:xacro="http://ros.org/wiki/xacro">
-    <xacro:arg name="laser_visual" default="false"/>
-    <xacro:arg name="imu_visual"   default="false"/>
-    <gazebo>
-        <plugin filename="libgazebo_ros_diff_drive.so" name="differential_drive_controller_front">
-            <rosDebugLevel>Debug</rosDebugLevel>
-            <publishWheelTF>True</publishWheelTF>
-            <publishTf>1</publishTf>
-            <publishWheelJointState>true</publishWheelJointState>
-            <alwaysOn>true</alwaysOn>
-            <updateRate>20.0</updateRate>
-            <leftJoint>l_wheel_joint</leftJoint>
-            <rightJoint>r_wheel_joint</rightJoint>
-            <wheelSeparation>0.076</wheelSeparation>
-            <wheelDiameter>0.034</wheelDiameter>
-            <broadcastTF>1</broadcastTF>
-            <wheelTorque>30</wheelTorque>
-            <wheelAcceleration>1.8</wheelAcceleration>
-            <commandTopic>cmd_vel</commandTopic>
-            <odometryFrame>odom</odometryFrame>
-            <odometryTopic>odom</odometryTopic>
-            <robotBaseFrame>base_link</robotBaseFrame>
-            <legacyMode>false</legacyMode>
-        </plugin>
-    </gazebo>
-    <gazebo reference="base_footprint">
-        <turnGravityOff>false</turnGravityOff>
-    </gazebo>
-    <gazebo reference="base_link">
-        <turnGravityOff>false</turnGravityOff>
-        <material>Gazebo/DarkYellow</material>
-    </gazebo>
-    <gazebo reference="l_wheel">
-        <mu1 value="1.0"/>
-        <mu2 value="1.0"/>
-        <kp value="10000000.0"/>
-        <kd value="1.0"/>
-        <fdir1 value="1 0 0"/>
-        <turnGravityOff>false</turnGravityOff>
-        <material>Gazebo/Black</material>
-    </gazebo>
-    <gazebo reference="r_wheel">
-        <mu1 value="1.0"/>
-        <mu2 value="1.0"/>
-        <kp value="10000000.0"/>
-        <kd value="1.0"/>
-        <fdir1 value="1 0 0"/>
-        <turnGravityOff>false</turnGravityOff>
-        <material>Gazebo/Black</material>
-    </gazebo>
-    <gazebo reference="caster_wheel">
-        <turnGravityOff>false</turnGravityOff>
-    </gazebo>
-    <gazebo>
-        <plugin name="imu_plugin" filename="libgazebo_ros_imu.so">
-            <alwaysOn>true</alwaysOn>
-            <bodyName>imu_link</bodyName>
-            <topicName>/imu</topicName>
-            <serviceName>/imu_service</serviceName>
-            <gaussianNoise>0.0</gaussianNoise>
-            <updateRate>100.0</updateRate>
-            <imu>
-                <noise>
-                    <type>gaussian</type>
-                    <rate>
-                        <mean>0.0</mean>
-                        <stddev>2e-4</stddev>
-                        <bias_mean>0.0000075</bias_mean>
-                        <bias_stddev>0.0000008</bias_stddev>
-                    </rate>
-                    <accel>
-                        <mean>0.0</mean>
-                        <stddev>1.7e-2</stddev>
-                        <bias_mean>0.1</bias_mean>
-                        <bias_stddev>0.001</bias_stddev>
-                    </accel>
-                </noise>
-            </imu>
-        </plugin>
-    </gazebo>
-    <gazebo reference="imu_link">
-        <sensor type="imu" name="imu">
-            <always_on>true</always_on>
-            <update_rate>50</update_rate>
-            <visualize>$(arg imu_visual)</visualize>
-        </sensor>
-        <material>Gazebo/Grey</material>
-    </gazebo>
-    <gazebo reference="base_scan">
-        <material>Gazebo/Grey</material>
-        <sensor type="ray" name="lds_lfcd_sensor">
-            <pose>0 0 0 0 0 0</pose>
-            <visualize>$(arg laser_visual)</visualize>
-            <update_rate>1800</update_rate>
-            <ray>
-                <scan>
-                    <horizontal>
-                        <samples>360</samples>
-                        <resolution>1</resolution>
-                        <min_angle>0.0</min_angle>
-                        <max_angle>6.28</max_angle>
-                    </horizontal>
-                </scan>
-                <range>
-                    <min>0.120</min>
-                    <max>3.5</max>
-                    <resolution>0.015</resolution>
-                </range>
-                <noise>
-                    <type>gaussian</type>
-                    <mean>0.0</mean>
-                    <stddev>0.01</stddev>
-                </noise>
-            </ray>
-            <plugin name="gazebo_ros_lds_lfcd_controller" filename="libgazebo_ros_laser.so">
-                <topicName>/scan</topicName>
-                <frameName>base_scan</frameName>
-            </plugin>
-        </sensor>
-    </gazebo>
-    <transmission name="l_wheel_joint_trans" >
-        <type>transmission_interface/SimpleTransmission</type>
-        <joint name="l_wheel_joint" />
-        <actuator name="l_wheel_joint_motor">
-            <hardwareInterface>EffortJointInterface</hardwareInterface>
-            <mechanicalReduction>1</mechanicalReduction>
-        </actuator>
-    </transmission>
-    <transmission name="r_wheel_joint_trans" >
-        <type>transmission_interface/SimpleTransmission</type>
-        <joint name="r_wheel_joint" />
-        <actuator name="r_wheel_joint_motor">
-            <hardwareInterface>EffortJointInterface</hardwareInterface>
-            <mechanicalReduction>1</mechanicalReduction>
-        </actuator>
-    </transmission>
+  <xacro:arg name="laser_visual" default="false"/>
+  <xacro:arg name="imu_visual"   default="false"/>
+  <gazebo>
+    <plugin name="candynamix_controller" filename="libgazebo_ros_diff_drive.so">
+      <commandTopic>cmd_vel</commandTopic>
+      <odometryTopic>odom</odometryTopic>
+      <odometryFrame>odom</odometryFrame>
+      <robotBaseFrame>base_footprint</robotBaseFrame>
+      <publishWheelTF>false</publishWheelTF>
+      <publishWheelJointState>true</publishWheelJointState>
+      <legacyMode>false</legacyMode>
+      <updateRate>100</updateRate>
+      <leftJoint>wheel_left_joint</leftJoint>
+      <rightJoint>wheel_right_joint</rightJoint>
+      <wheelSeparation>0.085</wheelSeparation>
+      <wheelDiameter>0.033</wheelDiameter>
+      <wheelAcceleration>1</wheelAcceleration>
+      <wheelTorque>10</wheelTorque>
+    </plugin>
+  </gazebo>
+  <gazebo reference="base_link">
+    <material><color rgba="${255/255} ${108/255} ${10/255} 1.0"/></material>
+  </gazebo>
+  <gazebo reference="wheel_left_link">
+    <mu1>10</mu1>
+    <mu2>10</mu2>
+    <kp>500000.0</kp>
+    <kd>10.0</kd>
+    <minDepth>0.001</minDepth>
+    <maxVel>0.1</maxVel>
+    <fdir1>1 0 0</fdir1>
+    <material>Gazebo/DarkGrey</material>
+  </gazebo>
+  <gazebo reference="wheel_right_link">
+    <mu1>10</mu1>
+    <mu2>10</mu2>
+    <kp>500000.0</kp>
+    <kd>10.0</kd>
+    <minDepth>0.001</minDepth>
+    <maxVel>0.1</maxVel>
+    <fdir1>1 0 0</fdir1>
+    <material>Gazebo/DarkGrey</material>
+  </gazebo>
+  <gazebo reference="caster_back_link">
+    <mu1>0.0</mu1>
+    <mu2>0.0</mu2>
+    <kp>1000000.0</kp>
+    <kd>100.0</kd>
+    <minDepth>0.001</minDepth>
+    <maxVel>1.0</maxVel>
+    <material>Gazebo/Grey</material>
+  </gazebo>
+  <gazebo>
+    <plugin name="imu_plugin" filename="libgazebo_ros_imu.so">
+      <alwaysOn>true</alwaysOn>
+      <bodyName>imu_link</bodyName>
+      <topicName>/imu</topicName>
+      <serviceName>/imu_service</serviceName>
+      <gaussianNoise>0.0</gaussianNoise>
+      <updateRate>100.0</updateRate>
+      <imu>
+        <noise>
+          <type>gaussian</type>
+          <rate>
+            <mean>0.0</mean>
+            <stddev>2e-4</stddev>
+            <bias_mean>0.0000075</bias_mean>
+            <bias_stddev>0.0000008</bias_stddev>
+          </rate>
+          <accel>
+            <mean>0.0</mean>
+            <stddev>1.7e-2</stddev>
+            <bias_mean>0.1</bias_mean>
+            <bias_stddev>0.001</bias_stddev>
+          </accel>
+        </noise>
+      </imu>
+    </plugin>
+  </gazebo>
+  <gazebo reference="imu_link">
+    <sensor type="imu" name="imu">
+      <always_on>true</always_on>
+      <update_rate>50</update_rate>
+      <visualize>$(arg imu_visual)</visualize>
+    </sensor>
+    <material>Gazebo/Grey</material>
+  </gazebo>
+  <gazebo reference="base_scan">
+    <material>Gazebo/DarkGrey</material>
+    <sensor type="ray" name="lds_lfcd_sensor">
+      <pose>0 0 0 0 0 0</pose>
+      <visualize>$(arg laser_visual)</visualize>
+      <update_rate>1800</update_rate>
+      <ray>
+        <scan>
+          <horizontal>
+            <samples>360</samples>
+            <resolution>1</resolution>
+            <min_angle>0.0</min_angle>
+            <max_angle>6.28</max_angle>
+          </horizontal>
+        </scan>
+        <range>
+          <min>0.120</min>
+          <max>3.5</max>
+          <resolution>0.015</resolution>
+        </range>
+        <noise>
+          <type>gaussian</type>
+          <mean>0.0</mean>
+          <stddev>0.01</stddev>
+        </noise>
+      </ray>
+      <plugin name="gazebo_ros_lds_lfcd_controller" filename="libgazebo_ros_laser.so">
+        <topicName>/scan</topicName>
+        <frameName>base_scan</frameName>
+      </plugin>
+    </sensor>
+  </gazebo>
 </robot>

File: canDynamix/candynamix_description/urdf/candynamix.urdf.xacro (robot description, xacro)
@@ -1,143 +1,197 @@
 <?xml version="1.0" ?>
 <robot name="candynamix" xmlns:xacro="http://ros.org/wiki/xacro">
-    <xacro:include filename="$(find candynamix_description)/urdf/common_properties.xacro"/>
-    <xacro:include filename="$(find candynamix_description)/urdf/candynamix.gazebo.xacro"/>
-    <link name="base_footprint">
-        <inertial>
-            <mass value="0.0001"/>
-            <origin xyz="0 0 0"/>
-            <inertia ixx="0.0001" ixy="0.0" ixz="0.0" iyy="0.0001" iyz="0.0" izz="0.0001"/>
-        </inertial>
-        <visual>
-            <origin rpy="0 0 0" xyz="0 0 0"/>
-            <geometry>
-                <box size="0.001 0.001 0.001"/>
-            </geometry>
-        </visual>
-    </link>
-    <link name="base_link">
-        <visual>
-            <!-- <origin xyz="-0.02 0 0.01" rpy="0 0 0" /> -->
-            <origin xyz="-0.0345 0.112 0.062" rpy="0 0 3.14"/>
-            <geometry>
-                <!-- <cylinder length="0.04" radius="0.06" /> -->
-                <mesh filename="package://candynamix_description/meshes/bases/candynamix_base.stl" scale="0.001 0.001 0.001"/>
-            </geometry>
-        </visual>
-        <collision>
-            <origin xyz="-0.01 0 0.015" rpy="0 0 0" />
-            <geometry>
-                <cylinder length="0.04" radius="0.055" />
-            </geometry>
-        </collision>
-        <inertial>
-            <origin xyz="0 0 0" rpy="0 0 0"/>
-            <mass value="5"/>
-                <inertia ixx="0.02" ixy="0.0" ixz="0.0" iyy="0.02" iyz="0.0" izz="0.05" />
-        </inertial>
-    </link>
-    <link name="l_wheel">
-        <visual>
-            <!-- <origin xyz="0 0 0" rpy="${90*3.14/180} 0 0" /> -->
-            <origin xyz="0 0 0" rpy="${-90*3.14/180} 0 0" />
-            <geometry>
-                <!-- <cylinder length="0.005" radius="0.02" /> -->
-                <mesh filename="package://candynamix_description/meshes/wheels/left_tire.stl" scale="0.001 0.001 0.001"/>
-            </geometry>
-        </visual>
-        <collision>
-            <origin xyz="0 0.005 0" rpy="${90*3.14/180} 0 0" />
-            <geometry>
-                <cylinder length="0.005" radius="0.017" />
-            </geometry>
-        </collision>
-        <inertial>
-            <origin xyz="0 0.0 0" rpy="0 0 0"/>
-            <mass value="2.5"/>
-            <inertia ixx="0.001" ixy="0.0" ixz="0.0" iyy="0.001" iyz="0.0" izz="0.002" />
-        </inertial>
-    </link>
-    <link name="r_wheel">
-        <visual>
-            <!-- <origin xyz="0 0 0" rpy="${90*3.14/180}0 0 0" /> -->
-            <origin xyz="0 0 0" rpy="${90*3.14/180} 0 0" />
-            <geometry>
-                <!-- <cylinder length="0.005" radius="0.02" /> -->
-                <mesh filename="package://candynamix_description/meshes/wheels/right_tire.stl" scale="0.001 0.001 0.001"/>
-            </geometry>
-        </visual>
-        <collision>
-            <origin xyz="0 -0.005 0" rpy="${90*3.14/180} 0 0" />
-            <geometry>
-                <cylinder length="0.005" radius="0.017" />
-            </geometry>
-        </collision>
-        <inertial>
-            <origin xyz="0 0 0" rpy="0 0 0"/>
-            <mass value="2.5"/>
-            <inertia ixx="0.001" ixy="0.0" ixz="0.0" iyy="0.001" iyz="0.0" izz="0.002" />
-        </inertial>
-    </link>
-    <link name="caster_wheel">
-        <visual>
-            <origin xyz="0 0 0" rpy="0 0 0" />
-            <geometry>
-                <sphere radius="0.008" />
-            </geometry>
-        </visual>
-        <collision>
-            <origin xyz="0 0 0" rpy="0 0 0" />
-            <geometry>
-                <sphere radius="0.01" />
-            </geometry>
-        </collision>
-        <inertial>
-            <origin xyz="0 0 0" rpy="0 0 0"/>
-            <mass value="0.5"/>
-            <inertia ixx="1.0" ixy="0.0" ixz="0.0" iyy="1.0" iyz="0.0" izz="1.0" />
-        </inertial>
-    </link>
-    <joint name="base_joint" type="fixed">
-        <parent link="base_footprint"/>
-        <child link="base_link"/>
-        <origin xyz="0 0 0.017" rpy="0 0 0"/>
-    </joint>
-    <joint name="l_wheel_joint" type="continuous">
-        <parent link="base_link"/>
-        <child link="l_wheel"/>
-        <axis xyz="0 1 0"/>
-        <origin xyz="0 0.038 0" rpy="0 0 0"/>
-        <joint_properties damping="0.0" friction="0.0"/>
-    </joint>
-    <joint name="r_wheel_joint" type="continuous">
-        <parent link="base_link"/>
-        <child link="r_wheel"/>
-        <axis xyz="0 1 0"/>
-        <origin xyz="0 -0.038 0" rpy="0 0 0"/>
-        <joint_properties damping="0.0" friction="0.0"/>
-    </joint>
-    <joint name="caster_joint" type="fixed">
-        <parent link="base_link"/>
-        <child link="caster_wheel"/>
-        <origin xyz="-0.055 0 -0.006" rpy="0 0 0"/>
-    </joint>
-    <link name="base_scan" type="fixed">
-        <visual>
-            <origin xyz="0 0 0" rpy="${90*3.14/180} 0 ${90*3.14/180} "/>
-            <geometry>
-                <mesh filename="package://candynamix_description/meshes/sensors/HC-SR04-UltrasonicSensor.stl" scale="0.001 0.001 0.001"/>
-            </geometry>
-        </visual>
-    </link>
-    <joint name="scan_joint" type="fixed">
-        <parent link="base_link"/>
-        <child link="base_scan"/>
-        <origin xyz="0.03 0 0.016" rpy="0 0 0 "/>
-    </joint>
-    <link name="imu_link"/>
-    <joint name="imu_joint" type="fixed">
-        <parent link="base_link"/>
-        <child link="imu_link"/>
-        <origin xyz="-0.032 0 0.068" rpy="0 0 0"/>
-    </joint>
+  <xacro:include filename="$(find candynamix_description)/urdf/common_properties.xacro"/>
+  <xacro:include filename="$(find candynamix_description)/urdf/candynamix.gazebo.xacro"/>
+  <link name="base_footprint"/>
+  <joint name="base_joint" type="fixed">
+    <parent link="base_footprint"/>
+    <child link="base_link"/>
+    <origin xyz="0 0 0" rpy="0 0 0"/>
+  </joint>
+  <link name="base_link">
+    <visual>
+	<origin xyz="-0.0345 0.112 0.077" rpy="0 0 3.14"/>
+      <geometry>
+        <mesh filename="package://candynamix_description/meshes/bases/candynamix_base.stl" scale="0.001 0.001 0.001"/>
+      </geometry>
+      <material name="orange"/>
+    </visual>
+    <collision>
+      <origin xyz="-0.01 0 0.035" rpy="0 0 0"/>
+      <geometry>
+        <cylinder length="0.05" radius="0.06"/>
+      </geometry>
+    </collision>
+    <inertial>
+      <origin xyz="0 0 0" rpy="0 0 0"/>
+      <mass value="1"/>
+      <inertia ixx="0.05" ixy="0.0" ixz="0.0"
+               iyy="0.05" iyz="0.0"
+               izz="0.05" />
+    </inertial>
+  </link>
+  <joint name="wheel_left_joint" type="continuous">
+    <parent link="base_link"/>
+    <child link="wheel_left_link"/>
+    <origin xyz="0 0.038 0.016" rpy="${M_PI*0.5} 1.57 1.57"/>
+    <axis xyz="0 1 0"/>
+  </joint>
+  <link name="wheel_left_link">
+    <visual>
+      <origin xyz="0 0 0" rpy="${-M_PI*0.5} 0 0"/>
+      <geometry>
+        <mesh filename="package://candynamix_description/meshes/wheels/left_tire.stl" scale="0.001 0.001 0.001"/>
+      </geometry>
+      <material name="dark"/>
+    </visual>
+    <collision>
+      <origin xyz="0 0.005 0" rpy="${-M_PI*0.5} 0 0"/>
+      <geometry>
+        <cylinder length="0.005" radius="0.018"/>
+      </geometry>
+    </collision>
+    <inertial>
+      <origin xyz="0 0 0" />
+      <mass value="0.01" />
+      <inertia ixx="0.05" ixy="0.0" ixz="0.0"
+               iyy="0.05" iyz="0.0"
+               izz="0.05" />
+    </inertial>
+  </link>
+  <joint name="wheel_right_joint" type="continuous">
+    <parent link="base_link"/>
+    <child link="wheel_right_link"/>
+    <origin xyz="0 -0.038 0.016" rpy="${-M_PI*0.5} -1.57 1.57"/>
+    <axis xyz="0 1 0"/>
+  </joint>
+  <link name="wheel_right_link">
+    <visual>
+      <origin xyz="0 0 0" rpy="${M_PI*0.5} 0 0"/>
+      <geometry>
+        <mesh filename="package://candynamix_description/meshes/wheels/right_tire.stl" scale="0.001 0.001 0.001"/>
+      </geometry>
+      <material name="dark"/>
+    </visual>
+    <collision>
+      <origin xyz="0 -0.005 0" rpy="${M_PI*0.5} 0 0"/>
+      <geometry>
+        <cylinder length="0.005" radius="0.018"/>
+      </geometry>
+    </collision>
+    <inertial>
+      <origin xyz="0 0 0" />
+      <mass value="0.01" />
+      <inertia ixx="0.05" ixy="0.0" ixz="0.0"
+               iyy="0.05" iyz="0.0"
+               izz="0.05" />
+    </inertial>
+  </link>
+  <joint name="caster_back_joint" type="fixed">
+    <parent link="base_link"/>
+    <child link="caster_back_link"/>
+    <origin xyz="-0.056 0 0.002" rpy="${-M_PI*0.5} 0 0"/>
+  </joint>
+  <link name="caster_back_link">
+    <collision>
+      <origin xyz="0 0 0" rpy="${M_PI*0.5} 0 0"/>
+      <geometry>
+        <cylinder length="0.005" radius="0.01"/>
+      </geometry>
+    </collision>
+    <inertial>
+      <origin xyz="0 0 0" />
+      <mass value="0.1" />
+      <inertia ixx="0.05" ixy="0.0" ixz="0.0"
+               iyy="0.05" iyz="0.0"
+               izz="0.05" />
+    </inertial>
+  </link>
+  <joint name="imu_joint" type="fixed">
+    <parent link="base_link"/>
+    <child link="imu_link"/>
+    <origin xyz="-0.032 0 0.068" rpy="0 0 0"/>
+  </joint>
+  <link name="imu_link"/>
+  <joint name="scan_joint" type="fixed">
+    <parent link="base_link"/>
+    <child link="base_scan"/>
+    <origin xyz="0.03 0 0.03" rpy="${M_PI*0.5} 0 0 "/>
+  </joint>
+  <link name="base_scan" type="fixed">
+    <visual>
+      <origin xyz="0 0 0" rpy="0 ${M_PI*0.5} 0 "/>
+      <geometry>
+        <mesh filename="package://candynamix_description/meshes/sensors/HC-SR04-UltrasonicSensor.stl" scale="0.001 0.001 0.001"/>
+      </geometry>
+      <material name="dark"/>
+    </visual>
+    <collision>
+      <origin xyz="0 0 0" rpy="5 10 60"/>
+      <geometry>
+        <cylinder length="0.003" radius="0.003"/>
+      </geometry>
+    </collision>
+    <inertial>
+      <mass value="0.01" />
+      <origin xyz="0 0 0" />
+      <inertia ixx="0.05" ixy="0.0" ixz="0.0"
+               iyy="0.05" iyz="0.0"
+               izz="0.05" />
+    </inertial>
+  </link>
+  <joint name="camera_joint" type="fixed">
+    <origin xyz="0.0605 -0.00 0.075" rpy="0 0 0"/>
+    <parent link="base_link"/>
+    <child link="camera_link"/>
+  </joint>
+  <link name="camera_link">
+    <visual>
+     <origin xyz="0 0 0" rpy="${M_PI*0.5} 0 ${M_PI*0.5}"/>
+      <geometry>
+       <mesh filename="package://candynamix_description/meshes/sensors/picamera.stl" scale="0.001 0.001 0.001" />
+      </geometry>
+      <material name="dark"/>
+    </visual>
+    <collision>
+      <origin xyz="0.003 0.065 0.010" rpy="0 0 0"/>
+      <geometry>
+        <box size="0.008 0.130 0.022"/>
+      </geometry>
+    </collision>
+    <!-- This inertial field needs doesn't contain reliable data!! -->
+ <!-- <inertial>
+      <mass value="0.564" />
+      <origin xyz="0 0 0" />
+      <inertia ixx="0.003881243" ixy="0.0" ixz="0.0"
+               iyy="0.000498940" iyz="0.0"
+               izz="0.003879257" />
+    </inertial>-->
+  </link>
+  <joint name="laser_joint" type="fixed">
+    <parent link="base_link"/>
+    <child link="laser_scan"/>
+    <origin xyz=" -0.025 0 0.120" rpy="0 0 0"/>
+  </joint>
+  <link name="laser_scan">
+    <visual>
+      <origin xyz="0 0 0.0" rpy="0 0 0"/>
+      <geometry>
+        <mesh filename="package://candynamix_description/meshes/sensors/lds.stl" scale="0.001 0.001 0.001"/>
+      </geometry>
+      <material name="dark"/>
+    </visual>
+    <collision>
+      <origin xyz="0 0 0" rpy="0 0 0"/>
+      <geometry>
+        <cylinder length="0.0408" radius="0.070"/>
+      </geometry>
+    </collision>
+    <inertial>
+      <mass value="0.01" />
+      <origin xyz="0 0 0" />
+      <inertia ixx="0.001" ixy="0.0" ixz="0.0"
+               iyy="0.001" iyz="0.0"
+               izz="0.001" />
+    </inertial>
+  </link>
 </robot>
